File: UccMicroDuino/UccMicroDuino.kicad_sch (KiCad schematic)
At the start: 14 parts, among them J1 Pcb USB Type A, J2 Header, U1 ATtiny85-20S

Commit message: 2634789-mi primer versionado con gitBash
Other:
- note added: "Circuito principal"
- note removed: "Main Circuit"
Changed lines of the file:
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@@
 		(comment 1 "proyectoBase2024")
 	)
-	(text "Main Circuit"
+	(text "Circuito principal"
 		(exclude_from_sim no)
 		(at 55.1942 140.9954 0)
